File: hardware/LEC001021.kicad_pcb (KiCad board)
At the start: 2 copper layers, 30 x 30 mm, 12 parts, among them J1 Screw_Terminal_01x02_blue

Commit message: Add OSHW logo
Parts:
- added REF**: OSHW-Logo2_7.3x6mm_SilkScreen, Symbol:OSHW-Logo2_7.3x6mm_SilkScreen, B.Cu at (129.5, 91.7)
